Commit message: 230218_complete

File: urdf/my_robot.xacro (robot description, xacro)
@@ -123,6 +123,6 @@
     <dynamics damping="1.0" friction="1.0"/>
   </joint>
- <!--camera-->
- <link name='camera'>
+  <!--camera-->
+  <link name='camera'>
     <pose>0 0 0 0 0 0</pose>
     <inertial>
@@ -182,4 +182,12 @@
     <axis xyz="0 1 0" rpy="0 0 0"/>
   </joint>
+  <!--RGBD-->
+  <joint name="camera_optical_joint" type="fixed">
+    <origin xyz="0 0 0" rpy="-1.5707 0 -1.5707"/>
+    <parent link="camera_link"/>
+    <child link="camera_link_optical"/>
+  </joint>
+  <link name="camera_link_optical">
+  </link>
   <!-- color is in last -->
   <gazebo reference="camera">
